File: schematic/epromemu.sch (KiCad schematic (older format))
At the start: 6 parts, among them J1 EPROM Connector, U1 Teensy4.1, U2 TXS0108EPW, U3 TXS0108EPW, U4 TXS0108EPW, U5 TXS0108EPW

Commit message: updates
Parts:
- removed U2, U3, U4, U5: TXS0108EPW, Package_SO:TSSOP-20_4.4x6.5mm_P0.65mm, symbol Logic_LevelTranslator:TXS0108EPW
- added U2, U3, U4, U5: 74HC245, Package_DIP:DIP-20_W7.62mm_Socket, symbol 74xx:74HC245
Connections:
- net +3V3: now also U3.20 (VCC), U4.20 (VCC), U5.20 (VCC)
- net +5V: now also J1.1 (Pin_1), U2.20 (VCC)
- net A0_3V3: now also U3.2 (A0)
- net A0_5V: now also U3.18 (B0)
- net A10_3V3: now also U4.4 (A2)
- net A10_5V: now also U4.16 (B2)
- net A11_3V3: now also U4.5 (A3)
- net A11_5V: now also U4.15 (B3)
- net A12_3V3: now also U4.6 (A4)
- net A12_5V: now also U4.14 (B4)
- net A13_3V3: now also U4.7 (A5)
- net A13_5V: now also U4.13 (B5)
- net A14_3V3: now also U4.8 (A6)
- net A14_5V: now also U4.12 (B6)
- net A15_3V3: now also U4.9 (A7)
- net A15_5V: now also U4.11 (B7)
- net A16_3V3: now also U5.2 (A0)
- net A16_5V: now also U5.18 (B0)
- net A17_3V3: now also U5.3 (A1)
- net A17_5V: now also U5.17 (B1)
- net A1_3V3: now also U3.3 (A1)
- net A1_5V: now also U3.17 (B1)
- net A2_3V3: now also U3.4 (A2)
- net A2_5V: now also U3.16 (B2)
- net A3_3V3: now also U3.5 (A3)
- net A3_5V: now also U3.15 (B3)
- net A4_3V3: now also U3.6 (A4)
- net A4_5V: now also U3.14 (B4)
- net A5_3V3: now also U3.7 (A5)
- net A5_5V: now also U3.13 (B5)
- net A6_3V3: now also U3.8 (A6)
- net A6_5V: now also U3.12 (B6)
- net A7_3V3: now also U3.9 (A7)
- net A7_5V: now also U3.11 (B7)
- net A8_3V3: now also U4.2 (A0)
- net A8_5V: now also U4.18 (B0)
- net A9_3V3: now also U4.3 (A1)
- net A9_5V: now also U4.17 (B1)
- net D0_3V3: now also U2.18 (B0)
- net D0_5V: now also U2.2 (A0)
- net D1_3V3: now also U2.17 (B1)
- net D1_5V: now also U2.3 (A1)
- net D2_3V3: now also U2.16 (B2)
- net D2_5V: now also U2.4 (A2)
- net D3_3V3: now also U2.15 (B3)
- net D3_5V: now also U2.5 (A3)
- net D4_3V3: now also U2.14 (B4)
- net D4_5V: now also U2.6 (A4)
- net D5_3V3: now also U2.13 (B5)
- net D5_5V: now also U2.7 (A5)
- net D6_3V3: now also U2.12 (B6)
- net D6_5V: now also U2.8 (A6)
- net D7_3V3: now also U2.11 (B7)
- net D7_5V: now also U2.9 (A7)
- net GND: now also U2.1 (A->B), U2.10 (GND), U3.1 (A->B), U3.10 (GND), U3.19 (CE), U4.1 (A->B), U4.10 (GND), U4.19 (CE), U5.1 (A->B), U5.10 (GND), U5.19 (CE); no longer J1.24 (Pin_24)
- net PGM_3V3: now reaches U1.25 (33_MCLK2)
- net PGM_3V3: now also U5.6 (A4)
- net CE_3V3: now reaches U1.26 (34_RX8)
- net CE_3V3: now also U5.5 (A3)
- net CE_5V: now reaches J1.22 (Pin_22)
- net CE_5V: now also U5.15 (B3)
- net PGM_5V: now reaches J1.31 (Pin_31)
- net PGM_5V: now also U5.14 (B4)
- new net OE_5V: J1.24 (Pin_24), U2.19 (CE)
- no-connect marks 53 -> 45

Commit message: update
Parts:
- added C2, C3, C4, C5: 0.1uf, Capacitor_THT:C_Disc_D5.0mm_W2.5mm_P5.00mm, symbol Device:C_Small
Connections:
- net +3V3: now also C3.1, C4.1, C5.1
- net +5V: now also C2.1
- net GND: now also C2.2, C3.2, C4.2, C5.2
Changed lines of the file:
@@
 	1    0    0    -1
 $EndComp
-Text GLabel 3300 1800 2    50   Input ~ 0
-D4_3V3
-Text GLabel 3300 2100 2    50   Input ~ 0
-D7_3V3
-Text GLabel 3300 1900 2    50   Input ~ 0
-D5_3V3
 Text GLabel 4250 1850 0    50   Input ~ 0
 D4_3V3
@@
 Text GLabel 4250 2250 0    50   Input ~ 0
 D0_3V3
-Text GLabel 3300 1400 2    50   Input ~ 0
-D0_3V3
-Text GLabel 3300 1600 2    50   Input ~ 0
-D2_3V3
 Text GLabel 4250 2350 0    50   Input ~ 0
 D2_3V3
 Text GLabel 4250 2450 0    50   Input ~ 0
 D1_3V3
-Text GLabel 3300 1500 2    50   Input ~ 0
-D1_3V3
 Text GLabel 4250 2650 0    50   Input ~ 0
 A0_3V3
-Text GLabel 2300 3550 0    50   Input ~ 0
-A0_3V3
-Text GLabel 2300 3650 0    50   Input ~ 0
-A1_3V3
 Text GLabel 4250 2750 0    50   Input ~ 0
 A1_3V3
@@
 Text GLabel 2300 1500 0    50   Input ~ 0
 D1_5V
-Text GLabel 3300 3550 2    50   Input ~ 0
-A0_5V
-Text GLabel 3300 3650 2    50   Input ~ 0
-A1_5V
 $Comp
 L power:GND #PWR0107
@@
 	1    5900 6650
 	-1   0    0    1
-$EndComp
-$Comp
-L power:+5V #PWR0114
-U 1 1 61B58CD7
-P 2800 1100
-F 0 "#PWR0114" H 2800 950 50  0001 C CNN
-F 1 "+5V" V 2815 1273 50  0000 C CNN
-F 2 "" H 2800 1100 50  0001 C CNN
-F 3 "" H 2800 1100 50  0001 C CNN
-	1    2800 1100
-	0    1    1    0
 $EndComp
 Text GLabel 5100 6350 0    50   Input ~ 0
@@
 Text GLabel 6450 2650 2    50   Input ~ 0
 A7_3V3
-Text GLabel 3300 2000 2    50   Input ~ 0
-D6_3V3
 Text GLabel 2300 2000 0    50   Input ~ 0
 D6_5V
@@
 Text GLabel 7350 1850 0    50   Input ~ 0
 A12_3V3
-Text GLabel 2300 3750 0    50   Input ~ 0
-A2_3V3
-Text GLabel 2300 3850 0    50   Input ~ 0
-A3_3V3
 Text GLabel 7350 1450 0    50   Input ~ 0
 A8_3V3
@@
 Text GLabel 8350 1850 2    50   Input ~ 0
 A12_5V
-Text GLabel 3300 3750 2    50   Input ~ 0
-A2_5V
-Text GLabel 3300 3850 2    50   Input ~ 0
-A3_5V
 Text GLabel 8350 1450 2    50   Input ~ 0
 A8_5V
@@
 Text GLabel 7350 2150 0    50   Input ~ 0
 A15_3V3
-Text GLabel 2300 4150 0    50   Input ~ 0
-A6_3V3
-Text GLabel 2300 4250 0    50   Input ~ 0
-A7_3V3
-Text GLabel 3300 1700 2    50   Input ~ 0
-D3_3V3
-Text GLabel 2300 3950 0    50   Input ~ 0
-A4_3V3
-Text GLabel 2300 4050 0    50   Input ~ 0
-A5_3V3
-Text GLabel 3300 4050 2    50   Input ~ 0
-A5_5V
-Text GLabel 3300 3950 2    50   Input ~ 0
-A4_5V
 Text GLabel 2300 1700 0    50   Input ~ 0
 D3_5V
-Text GLabel 3300 4250 2    50   Input ~ 0
-A7_5V
-Text GLabel 3300 4150 2    50   Input ~ 0
-A6_5V
 Text GLabel 8350 2150 2    50   Input ~ 0
 A15_5V
@@
 	1    7850 4850
 	1    0    0    -1
-$EndComp
-$Comp
-L power:+3.3V #PWR0108
-U 1 1 61C11FE4
-P 2800 3250
-F 0 "#PWR0108" H 2800 3100 50  0001 C CNN
-F 1 "+3.3V" V 2815 3378 50  0000 L CNN
-F 2 "" H 2800 3250 50  0001 C CNN
-F 3 "" H 2800 3250 50  0001 C CNN
-	1    2800 3250
-	0    1    1    0
-$EndComp
-$Comp
-L power:+3.3V #PWR0109
-U 1 1 61C12CCA
-P 7850 3250
-F 0 "#PWR0109" H 7850 3100 50  0001 C CNN
-F 1 "+3.3V" V 7865 3378 50  0000 L CNN
-F 2 "" H 7850 3250 50  0001 C CNN
-F 3 "" H 7850 3250 50  0001 C CNN
-	1    7850 3250
-	0    1    1    0
-$EndComp
-$Comp
-L power:+3.3V #PWR0110
-U 1 1 61C1329C
-P 7850 1150
-F 0 "#PWR0110" H 7850 1000 50  0001 C CNN
-F 1 "+3.3V" V 7865 1278 50  0000 L CNN
-F 2 "" H 7850 1150 50  0001 C CNN
-F 3 "" H 7850 1150 50  0001 C CNN
-	1    7850 1150
-	0    1    1    0
 $EndComp
 $Comp
@@
 	5900 6550 5900 6650
 Wire Wire Line
-	2800 2700 2150 2700
-Wire Wire Line
-	2150 2700 2150 2300
-Wire Wire Line
-	2150 2300 2300 2300
+	2800 2700 1950 2700
+Wire Wire Line
+	1950 2700 1950 2300
+Wire Wire Line
+	1950 2300 2300 2300
 Connection ~ 2800 2700
 Wire Wire Line
@@
 NoConn ~ 8350 3750
 NoConn ~ 7350 3750
+$Comp
+L power:GND #PWR0111
+U 1 1 61C3A75C
+P 1700 1300
+F 0 "#PWR0111" H 1700 1050 50  0001 C CNN
+F 1 "GND" H 1705 1127 50  0000 C CNN
+F 2 "" H 1700 1300 50  0001 C CNN
+F 3 "" H 1700 1300 50  0001 C CNN
+	1    1700 1300
+	1    0    0    -1
+$EndComp
+Wire Wire Line
+	1600 1100 1700 1100
+Connection ~ 1700 1100
+Wire Wire Line
+	1700 1100 2800 1100
+$Comp
+L power:GND #PWR0108
+U 1 1 61C52358
+P 1700 3450
+F 0 "#PWR0108" H 1700 3200 50  0001 C CNN
+F 1 "GND" H 1705 3277 50  0000 C CNN
+F 2 "" H 1700 3450 50  0001 C CNN
+F 3 "" H 1700 3450 50  0001 C CNN
+	1    1700 3450
+	1    0    0    -1
+$EndComp
+Wire Wire Line
+	1600 3250 1700 3250
+Connection ~ 1700 3250
+Wire Wire Line
+	1700 3250 2800 3250
+$Comp
+L power:GND #PWR0109
+U 1 1 61C5A8E3
+P 8950 1350
+F 0 "#PWR0109" H 8950 1100 50  0001 C CNN
+F 1 "GND" H 8955 1177 50  0000 C CNN
+F 2 "" H 8950 1350 50  0001 C CNN
+F 3 "" H 8950 1350 50  0001 C CNN
+	1    8950 1350
+	-1   0    0    -1
+$EndComp
+Wire Wire Line
+	9050 1150 8950 1150
+Connection ~ 8950 1150
+Wire Wire Line
+	8950 1150 7850 1150
+$Comp
+L power:+3.3V #PWR0110
+U 1 1 61C5A8EC
+P 9050 1150
+F 0 "#PWR0110" H 9050 1000 50  0001 C CNN
+F 1 "+3.3V" V 9065 1278 50  0000 L CNN
+F 2 "" H 9050 1150 50  0001 C CNN
+F 3 "" H 9050 1150 50  0001 C CNN
+	1    9050 1150
+	0    1    -1   0
+$EndComp
+$Comp
+L power:GND #PWR0115
+U 1 1 61C5BDC1
+P 8950 3450
+F 0 "#PWR0115" H 8950 3200 50  0001 C CNN
+F 1 "GND" H 8955 3277 50  0000 C CNN
+F 2 "" H 8950 3450 50  0001 C CNN
+F 3 "" H 8950 3450 50  0001 C CNN
+	1    8950 3450
+	-1   0    0    -1
+$EndComp
+Wire Wire Line
+	9050 3250 8950 3250
+Connection ~ 8950 3250
+Wire Wire Line
+	8950 3250 7850 3250
+$Comp
+L power:+3.3V #PWR0116
+U 1 1 61C5BDCA
+P 9050 3250
+F 0 "#PWR0116" H 9050 3100 50  0001 C CNN
+F 1 "+3.3V" V 9065 3378 50  0000 L CNN
+F 2 "" H 9050 3250 50  0001 C CNN
+F 3 "" H 9050 3250 50  0001 C CNN
+	1    9050 3250
+	0    1    -1   0
+$EndComp
+$Comp
+L Device:C_Small C2
+U 1 1 61C36AE0
+P 1700 1200
+F 0 "C2" H 1500 1200 50  0000 L CNN
+F 1 "0.1uf" H 1400 1100 50  0000 L CNN
+F 2 "Capacitor_THT:C_Disc_D5.0mm_W2.5mm_P5.00mm" H 1700 1200 50  0001 C CNN
+F 3 "~" H 1700 1200 50  0001 C CNN
+	1    1700 1200
+	1    0    0    -1
+$EndComp
+$Comp
+L Device:C_Small C3
+U 1 1 61C52352
+P 1700 3350
+F 0 "C3" H 1500 3350 50  0000 L CNN
+F 1 "0.1uf" H 1400 3250 50  0000 L CNN
+F 2 "Capacitor_THT:C_Disc_D5.0mm_W2.5mm_P5.00mm" H 1700 3350 50  0001 C CNN
+F 3 "~" H 1700 3350 50  0001 C CNN
+	1    1700 3350
+	1    0    0    -1
+$EndComp
+$Comp
+L Device:C_Small C4
+U 1 1 61C5A8DD
+P 8950 1250
+F 0 "C4" H 8850 1250 50  0000 R CNN
+F 1 "0.1uf" H 8850 1150 50  0000 R CNN
+F 2 "Capacitor_THT:C_Disc_D5.0mm_W2.5mm_P5.00mm" H 8950 1250 50  0001 C CNN
+F 3 "~" H 8950 1250 50  0001 C CNN
+	1    8950 1250
+	-1   0    0    -1
+$EndComp
+Text GLabel 3300 1700 2    50   Input ~ 0
+D3_3V3
+Text GLabel 3300 2000 2    50   Input ~ 0
+D6_3V3
+Text GLabel 3300 1500 2    50   Input ~ 0
+D1_3V3
+Text GLabel 3300 1600 2    50   Input ~ 0
+D2_3V3
+Text GLabel 3300 1400 2    50   Input ~ 0
+D0_3V3
+Text GLabel 3300 1900 2    50   Input ~ 0
+D5_3V3
+Text GLabel 3300 2100 2    50   Input ~ 0
+D7_3V3
+Text GLabel 3300 1800 2    50   Input ~ 0
+D4_3V3
+$Comp
+L power:+3.3V #PWR0113
+U 1 1 61C536FC
+P 1600 3250
+F 0 "#PWR0113" H 1600 3100 50  0001 C CNN
+F 1 "+3.3V" V 1615 3378 50  0000 L CNN
+F 2 "" H 1600 3250 50  0001 C CNN
+F 3 "" H 1600 3250 50  0001 C CNN
+	1    1600 3250
+	0    -1   -1   0
+$EndComp
+$Comp
+L power:+5V #PWR0114
+U 1 1 61B58CD7
+P 1600 1100
+F 0 "#PWR0114" H 1600 950 50  0001 C CNN
+F 1 "+5V" V 1615 1273 50  0000 C CNN
+F 2 "" H 1600 1100 50  0001 C CNN
+F 3 "" H 1600 1100 50  0001 C CNN
+	1    1600 1100
+	0    -1   -1   0
+$EndComp
+Text GLabel 3300 3950 2    50   Input ~ 0
+A4_5V
+Text GLabel 3300 4050 2    50   Input ~ 0
+A5_5V
+Text GLabel 3300 3850 2    50   Input ~ 0
+A3_5V
+Text GLabel 3300 3750 2    50   Input ~ 0
+A2_5V
+Text GLabel 3300 3650 2    50   Input ~ 0
+A1_5V
+Text GLabel 3300 3550 2    50   Input ~ 0
+A0_5V
+Text GLabel 2300 3550 0    50   Input ~ 0
+A0_3V3
+Text GLabel 2300 3650 0    50   Input ~ 0
+A1_3V3
+Text GLabel 2300 3750 0    50   Input ~ 0
+A2_3V3
+Text GLabel 2300 3850 0    50   Input ~ 0
+A3_3V3
+Text GLabel 2300 4150 0    50   Input ~ 0
+A6_3V3
+Text GLabel 2300 4250 0    50   Input ~ 0
+A7_3V3
+Text GLabel 2300 3950 0    50   Input ~ 0
+A4_3V3
+Text GLabel 2300 4050 0    50   Input ~ 0
+A5_3V3
+Text GLabel 3300 4150 2    50   Input ~ 0
+A6_5V
+Text GLabel 3300 4250 2    50   Input ~ 0
+A7_5V
+$Comp
+L Device:C_Small C5
+U 1 1 61C5BDBB
+P 8950 3350
+F 0 "C5" H 8850 3350 50  0000 R CNN
+F 1 "0.1uf" H 8850 3250 50  0000 R CNN
+F 2 "Capacitor_THT:C_Disc_D5.0mm_W2.5mm_P5.00mm" H 8950 3350 50  0001 C CNN
+F 3 "~" H 8950 3350 50  0001 C CNN
+	1    8950 3350
+	-1   0    0    -1
+$EndComp
 $EndSCHEMATC

Commit message: updates'
Connections:
- net +3V3: now also U4.1 (A->B), U5.1 (A->B)
- net A0_3V3: now also U3.18 (B0); no longer U3.2 (A0)
- net A0_5V: now also U3.2 (A0); no longer U3.18 (B0)
- net A10_3V3: now also U4.3 (A1); no longer U4.4 (A2)
- net A10_5V: now also U4.17 (B1); no longer U4.16 (B2)
- net A11_3V3: now also U4.2 (A0); no longer U4.5 (A3)
- net A11_5V: now also U4.18 (B0); no longer U4.15 (B3)
- net A12_3V3: now also U4.5 (A3); no longer U4.6 (A4)
- net A12_5V: now also U4.15 (B3); no longer U4.14 (B4)
- net A13_3V3: now also U4.4 (A2); no longer U4.7 (A5)
- net A13_5V: now also U4.16 (B2); no longer U4.13 (B5)
- net A14_3V3: now also U5.7 (A5); no longer U4.8 (A6)
- net A14_5V: now also U5.14 (B4); no longer U4.12 (B6)
- net A15_3V3: now also U5.6 (A4); no longer U4.9 (A7)
- net A15_5V: now also U5.13 (B5); no longer U4.11 (B7)
- net A16_3V3: now also U3.16 (B2); no longer U5.2 (A0)
- net A16_5V: now also U3.4 (A2); no longer U5.18 (B0)
- net A17_3V3: now also U3.15 (B3); no longer U5.3 (A1)
- net A17_5V: now also U3.5 (A3); no longer U5.17 (B1)
- net A1_3V3: now also U3.17 (B1); no longer U3.3 (A1)
- net A1_5V: now also U3.3 (A1); no longer U3.17 (B1)
- net A2_3V3: now also U4.6 (A4); no longer U3.4 (A2)
- net A2_5V: now also U4.14 (B4); no longer U3.16 (B2)
- net A3_3V3: now also U4.7 (A5); no longer U3.5 (A3)
- net A3_5V: now also U4.13 (B5); no longer U3.15 (B3)
- net A4_3V3: now also U5.3 (A1); no longer U3.6 (A4)
- net A4_5V: now also U5.17 (B1); no longer U3.14 (B4)
- net A5_3V3: now also U5.2 (A0); no longer U3.7 (A5)
- net A5_5V: now also U5.18 (B0); no longer U3.13 (B5)
- net A6_3V3: now also U5.5 (A3); no longer U3.8 (A6)
- net A6_5V: now also U5.15 (B3); no longer U3.12 (B6)
- net A7_3V3: now also U5.4 (A2); no longer U3.9 (A7)
- net A7_5V: now also U5.16 (B2); no longer U3.11 (B7)
- net A8_3V3: now also U4.8 (A6); no longer U4.2 (A0)
- net A8_5V: now also U4.12 (B6); no longer U4.18 (B0)
- net A9_3V3: now also U4.9 (A7); no longer U4.3 (A1)
- net A9_5V: now also U4.11 (B7); no longer U4.17 (B1)
- net CE_3V3: now also U5.8 (A6); no longer U5.5 (A3)
- net CE_5V: now also U5.12 (B6); no longer U5.15 (B3)
- net D0_3V3: now also U2.15 (B3); no longer U2.18 (B0)
- net D0_5V: now also U2.5 (A3); no longer U2.2 (A0)
- net D1_3V3: now also U2.13 (B5); no longer U2.17 (B1)
- net D1_5V: now also U2.7 (A5); no longer U2.3 (A1)
- net D2_3V3: now also U2.14 (B4); no longer U2.16 (B2)
- net D2_5V: now also U2.6 (A4); no longer U2.4 (A2)
- net D3_3V3: now also U2.11 (B7); no longer U2.15 (B3)
- net D3_5V: now also U2.9 (A7); no longer U2.5 (A3)
- net D4_3V3: now also U2.18 (B0); no longer U2.14 (B4)
- net D4_5V: now also U2.2 (A0); no longer U2.6 (A4)
- net D5_3V3: now also U2.16 (B2); no longer U2.13 (B5)
- net D5_5V: now also U2.4 (A2); no longer U2.7 (A5)
- net D7_3V3: now also U2.17 (B1); no longer U2.11 (B7)
- net D7_5V: now also U2.3 (A1); no longer U2.9 (A7)
- net GND: no longer U4.1 (A->B), U5.1 (A->B)
- net PGM_3V3: now also U5.9 (A7); no longer U5.6 (A4)
- net PGM_5V: now also U5.11 (B7); no longer U5.14 (B4)
- no-connect marks 45 -> 46
Other:
- moved on the sheet: C2, C3

Commit message: final?
Connections:
- net +3V3: now also U3.1 (A->B)
- net A0_3V3: now also U1.41 (19_A5_SCL), U4.6 (A4); no longer U1.16 (24_A10_TX6_SCL2), U3.18 (B0)
- net A0_5V: now also U4.14 (B4); no longer U3.2 (A0)
- net A10_3V3: now also U1.42 (20_A6_TX5_LRCLK1), U4.5 (A3); no longer U1.44 (22_A8_CTX1), U4.3 (A1)
- net A10_5V: now also U4.15 (B3); no longer U4.17 (B1)
- net A11_3V3: now also U1.43 (21_A7_RX5_BCLK1), U4.4 (A2); no longer U1.45 (23_A9_CRX1_MCLK1), U4.2 (A0)
- net A11_5V: now also U4.16 (B2); no longer U4.18 (B0)
- net A12_3V3: now also U1.30 (38_CS1_IN1), U5.7 (A5); no longer U1.42 (20_A6_TX5_LRCLK1), U4.5 (A3)
- net A12_5V: now also U5.13 (B5); no longer U4.15 (B3)
- net A13_3V3: now also U1.31 (39_MISO1_OUT1A), U5.6 (A4); no longer U1.43 (21_A7_RX5_BCLK1), U4.4 (A2)
- net A13_5V: now also U5.14 (B4); no longer U4.16 (B2)
- net A14_3V3: now also U1.18 (26_A12_MOSI1), U3.16 (B2); no longer U1.30 (38_CS1_IN1), U5.7 (A5)
- net A14_5V: now also U3.4 (A2); no longer U5.14 (B4)
- net A15_3V3: now also U1.19 (27_A13_SCK1), U3.15 (B3); no longer U1.31 (39_MISO1_OUT1A), U5.6 (A4)
- net A15_5V: now also U3.5 (A3); no longer U5.13 (B5)
- net A16_3V3: now also U1.16 (24_A10_TX6_SCL2), U3.18 (B0); no longer U1.18 (26_A12_MOSI1), U3.16 (B2)
- net A16_5V: now also U3.2 (A0); no longer U3.4 (A2)
- net A17_3V3: now also U1.17 (25_A11_RX6_SDA2), U3.17 (B1); no longer U1.19 (27_A13_SCK1), U3.15 (B3)
- net A17_5V: now also U3.3 (A1); no longer U3.5 (A3)
- net A1_3V3: now also U1.40 (18_A4_SDA), U4.7 (A5); no longer U1.17 (25_A11_RX6_SDA2), U3.17 (B1)
- net A1_5V: now also U4.13 (B5); no longer U3.3 (A1)
- net A2_3V3: now also U1.36 (14_A0_TX3_SPDIF_OUT), U5.3 (A1); no longer U1.41 (19_A5_SCL), U4.6 (A4)
- net A2_5V: now also U5.17 (B1); no longer U4.14 (B4)
- net A3_3V3: now also U1.37 (15_A1_RX3_SPDIF_IN), U5.2 (A0); no longer U1.40 (18_A4_SDA), U4.7 (A5)
- net A3_5V: now also U5.18 (B0); no longer U4.13 (B5)
- net A4_3V3: now also U1.32 (40_A16), U5.5 (A3); no longer U1.36 (14_A0_TX3_SPDIF_OUT), U5.3 (A1)
- net A4_5V: now also U5.15 (B3); no longer U5.17 (B1)
- net A5_3V3: now also U1.33 (41_A17), U5.4 (A2); no longer U1.37 (15_A1_RX3_SPDIF_IN), U5.2 (A0)
- net A5_5V: now also U5.16 (B2); no longer U5.18 (B0)
- net A6_3V3: now also U1.39 (17_A3_TX4_SDA1), U4.8 (A6); no longer U1.32 (40_A16), U5.5 (A3)
- net A6_5V: now also U4.12 (B6); no longer U5.15 (B3)
- net A7_3V3: now also U1.38 (16_A2_RX4_SCL1), U4.9 (A7); no longer U1.33 (41_A17), U5.4 (A2)
- net A7_5V: now also U4.11 (B7); no longer U5.16 (B2)
- net A8_3V3: now also U1.44 (22_A8_CTX1), U4.3 (A1); no longer U1.39 (17_A3_TX4_SDA1), U4.8 (A6)
- net A8_5V: now also U4.17 (B1); no longer U4.12 (B6)
- net A9_3V3: now also U1.45 (23_A9_CRX1_MCLK1), U4.2 (A0); no longer U1.38 (16_A2_RX4_SCL1), U4.9 (A7)
- net A9_5V: now also U4.18 (B0); no longer U4.11 (B7)
- net D0_3V3: now also U2.16 (B2); no longer U2.15 (B3)
- net D0_5V: now also U2.4 (A2); no longer U2.5 (A3)
- net D1_3V3: now also U2.14 (B4); no longer U2.13 (B5)
- net D1_5V: now also U2.6 (A4); no longer U2.7 (A5)
- net D2_3V3: now also U2.15 (B3); no longer U2.14 (B4)
- net D2_5V: now also U2.5 (A3); no longer U2.6 (A4)
- net D3_3V3: now also U2.13 (B5); no longer U2.11 (B7)
- net D3_5V: now also U2.7 (A5); no longer U2.9 (A7)
- net D4_3V3: now also U1.10 (8_TX2_IN1), U2.17 (B1); no longer U1.8 (6_OUT1D), U2.18 (B0)
- net D4_5V: now also U2.3 (A1); no longer U2.2 (A0)
- net D5_3V3: now also U1.9 (7_RX2_OUT1A), U2.18 (B0); no longer U1.11 (9_OUT1C), U2.16 (B2)
- net D5_5V: now also U2.2 (A0); no longer U2.4 (A2)
- net D6_3V3: now also U1.28 (36_CS), U2.11 (B7); no longer U1.24 (32_OUT1B), U2.12 (B6)
- net D6_5V: now also U2.9 (A7); no longer U2.8 (A6)
- net D7_3V3: now also U1.29 (37_CS), U2.12 (B6); no longer U1.10 (8_TX2_IN1), U2.17 (B1)
- net D7_5V: now also U2.8 (A6); no longer U2.3 (A1)
- net GND: no longer U3.1 (A->B)
- no-connect marks 46 -> 26
Other:
- moved on the sheet: C3, J1

Commit message: submitted v0.1
Connections:
- net +3V3: no longer U4.1 (A->B), U5.1 (A->B)
- net GND: now also U4.1 (A->B), U5.1 (A->B)
Changed lines of the file:
@@
 	9050 3250 8950 3250
 Connection ~ 8950 3250
-Wire Wire Line
-	8950 3250 8800 3250
 $Comp
 L power:+3.3V #PWR0116
@@
 	-1   0    0    -1
 $EndComp
-Wire Wire Line
-	7350 2350 7200 2350
-Wire Wire Line
-	7200 2350 7200 3000
-Wire Wire Line
-	8800 1150 7850 1150
-Wire Wire Line
-	8950 1150 8800 1150
-Connection ~ 8800 1150
-Wire Wire Line
-	7200 3000 8800 3000
-Wire Wire Line
-	8800 3000 8800 1150
-Wire Wire Line
-	7350 4450 7200 4450
-Wire Wire Line
-	7200 4450 7200 5100
-Wire Wire Line
-	7200 5100 8800 5100
-Wire Wire Line
-	8800 5100 8800 3250
-Connection ~ 8800 3250
-Wire Wire Line
-	8800 3250 7850 3250
 Wire Wire Line
 	1650 3250 1850 3250
@@
 	0    -1   -1   0
 $EndComp
+Wire Wire Line
+	7850 1150 8950 1150
+Wire Wire Line
+	7350 2350 7350 2450
+Connection ~ 7350 2450
+Wire Wire Line
+	7850 3250 8950 3250
+Wire Wire Line
+	7350 4450 7350 4550
+Connection ~ 7350 4550
 $EndSCHEMATC
