File: schematic/epromemu.kicad_pcb (KiCad board)
At the start: 2 copper layers, 6 parts, among them J1 EPROM Connector, U1 Teensy4.1, U2 TXS0108EPW, U3 TXS0108EPW, U4 TXS0108EPW, U5 TXS0108EPW

Commit message: updates
Parts:
- U2, U3, U4, U5: value TXS0108EPW -> 74HC245; footprint Package_SO:TSSOP-20_4.4x6.5mm_P0.65mm -> Package_DIP:DIP-20_W7.62mm_Socket
- moved U5 69.9 mm to (184.2, 85.1)
- moved U3 50.3 mm to (184.2, 49.5), turned to 90 degrees
- moved U2 46.2 mm to (149.9, 49.5), turned to 90 degrees
- moved J1 41.1 mm to (217.2, 44.5)
- moved U1 38.6 mm to (178.7, 64.3)
- moved U4 31.8 mm to (149.9, 85.1)
Connections:
- J1 pad 1: (no net) -> +5V
- J1 pad 22: (no net) -> CE_5V
- J1 pad 24: GND -> OE_5V
- J1 pad 31: (no net) -> PGM_5V
- U1 pad 25: (no net) -> PGM_3V3
- U1 pad 26: (no net) -> CE_3V3
- U2 pad 1: A1_3V3 -> GND
- U2 pad 10: (no net) -> GND
- U2 pad 11: GND -> D7_3V3
- U2 pad 12: D4_5V -> D6_3V3
- U2 pad 13: D7_5V -> D5_3V3
- U2 pad 14: D5_5V -> D4_3V3
- U2 pad 15: D0_5V -> D3_3V3
- U2 pad 16: D2_5V -> D2_3V3
- U2 pad 17: D1_5V -> D1_3V3
- U2 pad 18: A0_5V -> D0_3V3
- U2 pad 19: +5V -> OE_5V
- U2 pad 2: +3V3 -> D0_5V
- U2 pad 20: A1_5V -> +5V
- U2 pad 3: A0_3V3 -> D1_5V
- U2 pad 4: D1_3V3 -> D2_5V
- U2 pad 5: D2_3V3 -> D3_5V
- U2 pad 6: D0_3V3 -> D4_5V
- U2 pad 7: D5_3V3 -> D5_5V
- U2 pad 8: D7_3V3 -> D6_5V
- U2 pad 9: D4_3V3 -> D7_5V
- U3 pad 1: (no net) -> GND
- U3 pad 10: (no net) -> GND
- U3 pad 11: GND -> A7_5V
- U3 pad 12: A16_5V -> A6_5V
- U3 pad 13: A17_5V -> A5_5V
- U3 pad 14: D6_5V -> A4_5V
- U3 pad 15: (no net) -> A3_5V
- U3 pad 16: (no net) -> A2_5V
- U3 pad 17: (no net) -> A1_5V
- U3 pad 18: (no net) -> A0_5V
- U3 pad 19: +5V -> GND
- U3 pad 2: +3V3 -> A0_3V3
- U3 pad 20: (no net) -> +3V3
- U3 pad 3: (no net) -> A1_3V3
- U3 pad 4: (no net) -> A2_3V3
- U3 pad 5: (no net) -> A3_3V3
- U3 pad 6: (no net) -> A4_3V3
- U3 pad 7: D6_3V3 -> A5_3V3
- U3 pad 8: A17_3V3 -> A6_3V3
- U3 pad 9: A16_3V3 -> A7_3V3
- U4 pad 1: A5_3V3 -> GND
- U4 pad 10: (no net) -> GND
- U4 pad 11: GND -> A15_5V
- U4 pad 12: (no net) -> A14_5V
- U4 pad 13: A14_5V -> A13_5V
- U4 pad 14: A15_5V -> A12_5V
- U4 pad 15: A6_5V -> A11_5V
- U4 pad 16: A7_5V -> A10_5V
- U4 pad 17: D3_5V -> A9_5V
- U4 pad 18: A4_5V -> A8_5V
- U4 pad 19: +5V -> GND
- U4 pad 2: +3V3 -> A8_3V3
- U4 pad 20: A5_5V -> +3V3
- U4 pad 3: A4_3V3 -> A9_3V3
- U4 pad 4: D3_3V3 -> A10_3V3
- U4 pad 5: A7_3V3 -> A11_3V3
- U4 pad 6: A6_3V3 -> A12_3V3
- U4 pad 7: A15_3V3 -> A13_3V3
- U4 pad 9: (no net) -> A15_3V3
- U5 pad 1: A11_3V3 -> GND
- U5 pad 10: (no net) -> GND
- U5 pad 11: GND -> (no net)
- U5 pad 12: A9_5V -> (no net)
- U5 pad 13: A8_5V -> (no net)
- U5 pad 14: A3_5V -> PGM_5V
- U5 pad 15: A2_5V -> CE_5V
- U5 pad 16: A12_5V -> (no net)
- U5 pad 17: A13_5V -> A17_5V
- U5 pad 18: A10_5V -> A16_5V
- U5 pad 19: +5V -> GND
- U5 pad 2: +3V3 -> A16_3V3
- U5 pad 20: A11_5V -> +3V3
- U5 pad 3: A10_3V3 -> A17_3V3
- U5 pad 4: A13_3V3 -> (no net)
- U5 pad 5: A12_3V3 -> CE_3V3
- U5 pad 6: A2_3V3 -> PGM_3V3
- U5 pad 7: A3_3V3 -> (no net)
- U5 pad 8: A8_3V3 -> (no net)
- U5 pad 9: A9_3V3 -> (no net)
Routing:
- net GND: track 170.5 -> 0.00 mm, vias 1 -> 0
- net +5V: track 158.4 -> 0.00 mm, vias 2 -> 0
- net +3V3: track 98.3 -> 0.00 mm, vias 2 -> 0
- net D5_5V: track 85.4 -> 0.00 mm, vias 1 -> 0
- net D1_5V: track 79.7 -> 0.00 mm
- net A9_5V: track 78.8 -> 0.00 mm, vias 1 -> 0
- net D7_5V: track 78.0 -> 0.00 mm, vias 1 -> 0
- net A16_5V: track 74.9 -> 0.00 mm
- net A13_5V: track 74.4 -> 0.00 mm, vias 1 -> 0
- net A0_5V: track 72.4 -> 0.00 mm
- net A11_5V: track 71.2 -> 0.00 mm, vias 1 -> 0
- net D4_5V: track 70.7 -> 0.00 mm
- net A8_5V: track 69.5 -> 0.00 mm, vias 1 -> 0
- net A10_5V: track 68.8 -> 0.00 mm, vias 1 -> 0
- net D2_5V: track 68.6 -> 0.00 mm
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Other:
- board outline added: 81.3 x 52.1 mm
- board text added: "EPROM Emulator v1.0 Brian Peek"

Commit message: update
Parts:
- added C2: 0.1uf, Capacitor_THT:C_Disc_D5.0mm_W2.5mm_P5.00mm, F.Cu at (146.6, 45.2)
- added C3: 0.1uf, Capacitor_THT:C_Disc_D5.0mm_W2.5mm_P5.00mm, F.Cu at (180.8, 45.2)
- added C4: 0.1uf, Capacitor_THT:C_Disc_D5.0mm_W2.5mm_P5.00mm, F.Cu at (146.6, 79.0)
- added C5: 0.1uf, Capacitor_THT:C_Disc_D5.0mm_W2.5mm_P5.00mm, F.Cu at (180.8, 79.0)
- moved U2 1.78 mm to (149.9, 51.3)
- moved U3 1.78 mm to (184.2, 51.3)
- moved J1 1.27 mm to (215.9, 44.5)
Other:
- board size 81.3 x 52.1 mm -> 79.2 x 47.2 mm
- board text removed: "EPROM Emulator v1.0 Brian Peek"

Commit message: updates'
Parts:
- moved C5 35.9 mm to (181.0, 43.1)
- moved C4 35.9 mm to (146.6, 43.1)
- moved U4 35.7 mm to (149.9, 49.4)
- moved U5 35.7 mm to (184.2, 49.4)
- moved U2 35.3 mm to (149.9, 86.6)
- moved U3 35.3 mm to (184.2, 86.6)
- moved C2 35.1 mm to (146.7, 80.3)
- moved C3 35.1 mm to (180.8, 80.3)
- moved J1 0.98 mm to (215.6, 45.4)
Connections:
- U2 pad 11: D7_3V3 -> D3_3V3
- U2 pad 13: D5_3V3 -> D1_3V3
- U2 pad 14: D4_3V3 -> D2_3V3
- U2 pad 15: D3_3V3 -> D0_3V3
- U2 pad 16: D2_3V3 -> D5_3V3
- U2 pad 17: D1_3V3 -> D7_3V3
- U2 pad 18: D0_3V3 -> D4_3V3
- U2 pad 2: D0_5V -> D4_5V
- U2 pad 3: D1_5V -> D7_5V
- U2 pad 4: D2_5V -> D5_5V
- U2 pad 5: D3_5V -> D0_5V
- U2 pad 6: D4_5V -> D2_5V
- U2 pad 7: D5_5V -> D1_5V
- U2 pad 9: D7_5V -> D3_5V
- U3 pad 11: A7_5V -> (no net)
- U3 pad 12: A6_5V -> (no net)
- U3 pad 13: A5_5V -> (no net)
- U3 pad 14: A4_5V -> (no net)
- U3 pad 15: A3_5V -> A17_3V3
- U3 pad 16: A2_5V -> A16_3V3
- U3 pad 17: A1_5V -> A1_3V3
- U3 pad 18: A0_5V -> A0_3V3
- U3 pad 2: A0_3V3 -> A0_5V
- U3 pad 3: A1_3V3 -> A1_5V
- U3 pad 4: A2_3V3 -> A16_5V
- U3 pad 5: A3_3V3 -> A17_5V
- U3 pad 6: A4_3V3 -> (no net)
- U3 pad 7: A5_3V3 -> (no net)
- U3 pad 8: A6_3V3 -> (no net)
- U3 pad 9: A7_3V3 -> (no net)
- U4 pad 1: GND -> +3V3
- U4 pad 11: A15_5V -> A9_5V
- U4 pad 12: A14_5V -> A8_5V
- U4 pad 13: A13_5V -> A3_5V
- U4 pad 14: A12_5V -> A2_5V
- U4 pad 15: A11_5V -> A12_5V
- U4 pad 16: A10_5V -> A13_5V
- U4 pad 17: A9_5V -> A10_5V
- U4 pad 18: A8_5V -> A11_5V
- U4 pad 2: A8_3V3 -> A11_3V3
- U4 pad 3: A9_3V3 -> A10_3V3
- U4 pad 4: A10_3V3 -> A13_3V3
- U4 pad 5: A11_3V3 -> A12_3V3
- U4 pad 6: A12_3V3 -> A2_3V3
- U4 pad 7: A13_3V3 -> A3_3V3
- U4 pad 8: A14_3V3 -> A8_3V3
- U4 pad 9: A15_3V3 -> A9_3V3
- U5 pad 1: GND -> +3V3
- U5 pad 11: (no net) -> PGM_5V
- U5 pad 12: (no net) -> CE_5V
- U5 pad 13: (no net) -> A15_5V
- U5 pad 14: PGM_5V -> A14_5V
- U5 pad 15: CE_5V -> A6_5V
- U5 pad 16: (no net) -> A7_5V
- U5 pad 17: A17_5V -> A4_5V
- U5 pad 18: A16_5V -> A5_5V
- U5 pad 2: A16_3V3 -> A5_3V3
- U5 pad 3: A17_3V3 -> A4_3V3
- U5 pad 4: (no net) -> A7_3V3
- U5 pad 5: CE_3V3 -> A6_3V3
- U5 pad 6: PGM_3V3 -> A15_3V3
- U5 pad 7: (no net) -> A14_3V3
- U5 pad 8: (no net) -> CE_3V3
- U5 pad 9: (no net) -> PGM_3V3
Other:
- board size 79.2 x 47.2 mm -> 82.3 x 54.1 mm
- board text added: "EPROM Emulator v1.0 Brian Peek"

Commit message: final?
Connections:
- U1 pad 10: D7_3V3 -> D4_3V3
- U1 pad 11: D5_3V3 -> (no net)
- U1 pad 16: A0_3V3 -> A16_3V3
- U1 pad 17: A1_3V3 -> A17_3V3
- U1 pad 18: A16_3V3 -> A14_3V3
- U1 pad 19: A17_3V3 -> A15_3V3
- U1 pad 24: D6_3V3 -> (no net)
- U1 pad 28: (no net) -> D6_3V3
- U1 pad 29: (no net) -> D7_3V3
- U1 pad 30: A14_3V3 -> A12_3V3
- U1 pad 31: A15_3V3 -> A13_3V3
- U1 pad 32: A6_3V3 -> A4_3V3
- U1 pad 33: A7_3V3 -> A5_3V3
- U1 pad 36: A4_3V3 -> A2_3V3
- U1 pad 37: A5_3V3 -> A3_3V3
- U1 pad 38: A9_3V3 -> A7_3V3
- U1 pad 39: A8_3V3 -> A6_3V3
- U1 pad 40: A3_3V3 -> A1_3V3
- U1 pad 41: A2_3V3 -> A0_3V3
- U1 pad 42: A12_3V3 -> A10_3V3
- U1 pad 43: A13_3V3 -> A11_3V3
- U1 pad 44: A10_3V3 -> A8_3V3
- U1 pad 45: A11_3V3 -> A9_3V3
- U1 pad 8: D4_3V3 -> (no net)
- U1 pad 9: (no net) -> D5_3V3
- U2 pad 11: D3_3V3 -> D6_3V3
- U2 pad 12: D6_3V3 -> D7_3V3
- U2 pad 13: D1_3V3 -> D3_3V3
- U2 pad 14: D2_3V3 -> D1_3V3
- U2 pad 15: D0_3V3 -> D2_3V3
- U2 pad 16: D5_3V3 -> D0_3V3
- U2 pad 17: D7_3V3 -> D4_3V3
- U2 pad 18: D4_3V3 -> D5_3V3
- U2 pad 2: D4_5V -> D5_5V
- U2 pad 3: D7_5V -> D4_5V
- U2 pad 4: D5_5V -> D0_5V
- U2 pad 5: D0_5V -> D2_5V
- U2 pad 6: D2_5V -> D1_5V
- U2 pad 7: D1_5V -> D3_5V
- U2 pad 8: D6_5V -> D7_5V
- U2 pad 9: D3_5V -> D6_5V
- U3 pad 1: GND -> +3V3
- U3 pad 15: A17_3V3 -> A15_3V3
- U3 pad 16: A16_3V3 -> A14_3V3
- U3 pad 17: A1_3V3 -> A17_3V3
- U3 pad 18: A0_3V3 -> A16_3V3
- U3 pad 2: A0_5V -> A16_5V
- U3 pad 3: A1_5V -> A17_5V
- U3 pad 4: A16_5V -> A14_5V
- U3 pad 5: A17_5V -> A15_5V
- U4 pad 11: A9_5V -> A7_5V
- U4 pad 12: A8_5V -> A6_5V
- U4 pad 13: A3_5V -> A1_5V
- U4 pad 14: A2_5V -> A0_5V
- U4 pad 15: A12_5V -> A10_5V
- U4 pad 16: A13_5V -> A11_5V
- U4 pad 17: A10_5V -> A8_5V
- U4 pad 18: A11_5V -> A9_5V
- U4 pad 2: A11_3V3 -> A9_3V3
- U4 pad 3: A10_3V3 -> A8_3V3
- U4 pad 4: A13_3V3 -> A11_3V3
- U4 pad 5: A12_3V3 -> A10_3V3
- U4 pad 6: A2_3V3 -> A0_3V3
- U4 pad 7: A3_3V3 -> A1_3V3
- U4 pad 8: A8_3V3 -> A6_3V3
- U4 pad 9: A9_3V3 -> A7_3V3
- U5 pad 13: A15_5V -> A12_5V
- U5 pad 14: A14_5V -> A13_5V
- U5 pad 15: A6_5V -> A4_5V
- U5 pad 16: A7_5V -> A5_5V
- U5 pad 17: A4_5V -> A2_5V
- U5 pad 18: A5_5V -> A3_5V
- U5 pad 2: A5_3V3 -> A3_3V3
- U5 pad 3: A4_3V3 -> A2_3V3
- U5 pad 4: A7_3V3 -> A5_3V3
- U5 pad 5: A6_3V3 -> A4_3V3
- U5 pad 6: A15_3V3 -> A13_3V3
- U5 pad 7: A14_3V3 -> A12_3V3
Routing:
- net GND: track 0.00 -> 199.0 mm
- net +5V: track 0.00 -> 128.5 mm
- net +3V3: track 0.00 -> 125.5 mm
- net D4_5V: track 0.00 -> 85.0 mm
- net D5_5V: track 0.00 -> 80.6 mm
- net A8_5V: track 0.00 -> 80.0 mm
- net A9_5V: track 0.00 -> 73.0 mm
- net OE_5V: track 0.00 -> 72.6 mm, vias 0 -> 1
- net A0_5V: track 0.00 -> 71.6 mm, vias 0 -> 1
- net A1_5V: track 0.00 -> 69.6 mm
- net D3_5V: track 0.00 -> 68.6 mm
- net A11_5V: track 0.00 -> 67.9 mm
- net D0_5V: track 0.00 -> 65.5 mm
- net A10_5V: track 0.00 -> 63.5 mm
- net D2_5V: track 0.00 -> 62.2 mm
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Other:
- board size 82.3 x 54.1 mm -> 80.5 x 53.6 mm
- net class Default: clearance 0.2 -> 0.1524; trace_width 0.25 -> 0.1524; via_dia 0.8 -> 0.6858; via_drill 0.4 -> 0.3302
- rule pad_to_mask_clearance: 0 -> 0.0508
- rule trace_clearance: 0.2 -> 0.1524
- rule trace_min: 0.2 -> 0.1524
- rule via_min_drill: 0.3 -> 0.254
- rule via_min_size: 0.4 -> 0.508
- board text added: "EPROM Emulator v0.1 - Brian Peek"
- board text removed: "EPROM Emulator v1.0 Brian Peek"

Commit message: submitted v0.1
Connections:
- U4 pad 1: +3V3 -> GND
- U5 pad 1: +3V3 -> GND
Routing:
- net PGM_5V: track 55.0 -> 11.2 mm
- net +5V: track 128.5 -> 87.3 mm
- net A10_5V: track 63.5 -> 89.2 mm
- net A0_5V: track 71.6 -> 91.0 mm, vias 1 -> 0
- net D4_5V: track 85.0 -> 65.7 mm
- net A14_5V: track 28.8 -> 47.7 mm, vias 1 -> 0
- net A13_5V: track 54.0 -> 36.5 mm
- net +3V3: track 125.5 -> 108.5 mm
- net A17_5V: track 31.3 -> 48.2 mm
- net D3_5V: track 68.6 -> 52.0 mm
- net CE_5V: track 29.1 -> 44.7 mm
- net A1_5V: track 69.6 -> 84.8 mm
- net A8_5V: track 80.0 -> 65.1 mm
- net A4_5V: track 54.3 -> 40.4 mm
- net D5_5V: track 80.6 -> 66.8 mm
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
Commit message: update to v6
Parts:
- moved U4 49.8 mm to (112.6, 82.5)
- moved C2 49.8 mm to (109.4, 113.3)
- moved C3 49.8 mm to (143.6, 113.3)
- moved C4 49.8 mm to (109.3, 76.1)
- moved C5 49.8 mm to (143.7, 76.1)
- moved J1 49.8 mm to (178.4, 78.5)
- moved U2 49.8 mm to (112.6, 119.7)
- moved U5 49.8 mm to (146.9, 82.5)
- moved U1 49.8 mm to (141.4, 97.4)
- moved U3 49.8 mm to (146.9, 119.7)
Connections:
- U1 pad 11: (no net) -> unconnected-(U1-Pad11)
- U1 pad 2: (no net) -> unconnected-(U1-Pad2)
- U1 pad 20: (no net) -> unconnected-(U1-Pad20)
- U1 pad 21: (no net) -> unconnected-(U1-Pad21)
- U1 pad 22: (no net) -> unconnected-(U1-Pad22)
- U1 pad 23: (no net) -> unconnected-(U1-Pad23)
- U1 pad 24: (no net) -> unconnected-(U1-Pad24)
- U1 pad 27: (no net) -> unconnected-(U1-Pad27)
- U1 pad 3: (no net) -> unconnected-(U1-Pad3)
- U1 pad 34: (no net) -> unconnected-(U1-Pad34)
- U1 pad 4: (no net) -> unconnected-(U1-Pad4)
- U1 pad 46: (no net) -> unconnected-(U1-Pad46)
- U1 pad 47: (no net) -> unconnected-(U1-Pad47)
- U1 pad 48: (no net) -> unconnected-(U1-Pad48)
- U1 pad 5: (no net) -> unconnected-(U1-Pad5)
- U1 pad 6: (no net) -> unconnected-(U1-Pad6)
- U1 pad 7: (no net) -> unconnected-(U1-Pad7)
- U1 pad 8: (no net) -> unconnected-(U1-Pad8)
- U3 pad 11: (no net) -> unconnected-(U3-Pad11)
- U3 pad 12: (no net) -> unconnected-(U3-Pad12)
- U3 pad 13: (no net) -> unconnected-(U3-Pad13)
- U3 pad 14: (no net) -> unconnected-(U3-Pad14)
- U3 pad 6: (no net) -> unconnected-(U3-Pad6)
- U3 pad 7: (no net) -> unconnected-(U3-Pad7)
- U3 pad 8: (no net) -> unconnected-(U3-Pad8)
- U3 pad 9: (no net) -> unconnected-(U3-Pad9)
Other:
- net class Default removed

Commit message: v0.2 updates
Connections:
- U1 pad 20: unconnected-(U1-Pad20) -> OE_3V3
- U1 pad 22: unconnected-(U1-Pad22) -> CE_3V3
- U1 pad 23: unconnected-(U1-Pad23) -> PGM_3V3
- U1 pad 25: PGM_3V3 -> unconnected-(U1-Pad25)
- U1 pad 26: CE_3V3 -> unconnected-(U1-Pad26)
- U2 pad 19: OE_5V -> CE_5V
- U3 pad 11: unconnected-(U3-Pad11) -> PGM_3V3
- U3 pad 9: unconnected-(U3-Pad9) -> PGM_5V
- U5 pad 11: PGM_5V -> OE_5V
- U5 pad 9: PGM_3V3 -> OE_3V3
Routing:
- net CE_5V: track 44.7 -> 118.9 mm
- net PGM_5V: track 11.2 -> 57.1 mm
- net OE_5V: track 70.3 -> 33.5 mm
- net +5V: track 87.3 -> 113.5 mm
- net OE_3V3: track 0.00 -> 25.3 mm, vias 0 -> 1
- net A0_5V: track 91.0 -> 67.1 mm
- net A1_5V: track 84.8 -> 63.7 mm
- net +3V3: track 108.5 -> 125.7 mm
- net A10_5V: track 89.2 -> 72.1 mm
- net A2_5V: track 55.9 -> 39.5 mm
- net A17_5V: track 48.2 -> 64.1 mm
- net CE_3V3: track 8.70 -> 23.2 mm, vias 0 -> 1
- net A13_5V: track 36.5 -> 22.1 mm
- net A16_5V: track 55.6 -> 69.2 mm
- net A3_5V: track 55.9 -> 42.6 mm
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Other:
- board text added: "EPROM Emulator v0.2 - Brian Peek"
- board text removed: "EPROM Emulator v0.1 - Brian Peek"

Commit message: v0.2 in progress...
Parts:
- moved J1 37.6 mm to (181.0, 116.0), turned to 180 degrees
Connections:
- J1 pad 31: PGM_5V -> A18_5V
- U1 pad 20: OE_3V3 -> A18_3V3
- U1 pad 21: unconnected-(U1-Pad21) -> CE_OE
- U1 pad 22: CE_3V3 -> OE_3V3
- U1 pad 23: PGM_3V3 -> CE_3V3
- U2 pad 19: CE_5V -> CE_OE
- U3 pad 11: PGM_3V3 -> CE_3V3
- U3 pad 12: unconnected-(U3-Pad12) -> OE_3V3
- U3 pad 14: unconnected-(U3-Pad14) -> A18_3V3
- U3 pad 6: unconnected-(U3-Pad6) -> A18_5V
- U3 pad 8: unconnected-(U3-Pad8) -> OE_5V
- U3 pad 9: PGM_5V -> CE_5V
- U5 pad 11: OE_5V -> unconnected-(U5-Pad11)
- U5 pad 12: CE_5V -> unconnected-(U5-Pad12)
- U5 pad 8: CE_3V3 -> unconnected-(U5-Pad8)
- U5 pad 9: OE_3V3 -> unconnected-(U5-Pad9)
Routing:
- net GND: track 197.5 -> 0.00 mm
- net +3V3: track 125.7 -> 0.00 mm
- net CE_5V: track 118.9 -> 0.00 mm
- net +5V: track 113.5 -> 0.00 mm
- net D4_5V: track 74.1 -> 0.00 mm
- net A10_5V: track 72.1 -> 0.00 mm
- net A9_5V: track 70.4 -> 0.00 mm, vias 1 -> 0
- net A16_5V: track 69.2 -> 0.00 mm
- net A8_5V: track 68.8 -> 0.00 mm
- net D5_5V: track 68.1 -> 0.00 mm
- net A0_5V: track 67.1 -> 0.00 mm
- net D2_5V: track 66.8 -> 0.00 mm
- net A11_5V: track 66.8 -> 0.00 mm
- net D0_5V: track 66.5 -> 0.00 mm
- net A17_5V: track 64.1 -> 0.00 mm
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