File: schematic_old/epromemu.kicad_sch (KiCad schematic)
At the start: 19 parts, among them J3 EPROM Connector, U1 Teensy4.1, U2 74HC245, U3 74HC245, U4 74HC245, U5 74HC245, U6 74HC32

Commit message: Rev C schem/pcb
Parts:
- removed JP2: A17, Connector_PinHeader_2.54mm:PinHeader_1x03_P2.54mm_Vertical, symbol Jumper:Jumper_3_Open
- removed JP3: A13, Connector_PinHeader_2.54mm:PinHeader_1x03_P2.54mm_Vertical, symbol Jumper:Jumper_3_Open
- added J1: EPROM Connector, Connector_PinHeader_2.54mm:PinHeader_2x12_P2.54mm_Vertical, symbol Connector_Generic:Conn_02x12_Counter_Clockwise
- added J2: EPROM Connector, Connector_PinHeader_2.54mm:PinHeader_2x14_P2.54mm_Vertical, symbol Connector_Generic:Conn_02x14_Counter_Clockwise
Connections:
- net +3V3: now also U3.1 (A->B); no longer U4.1 (A->B), U5.1 (A->B)
- net +5V: no longer U2.1 (A->B)
- net A0_3V3: now also U4.6 (A4); no longer U4.15 (B3)
- net A0_5V: now also U4.14 (B4), J1.8 (Pin_8), J2.10 (Pin_10); no longer U4.5 (A3)
- net A10_3V3: now also U4.5 (A3); no longer U3.9 (A7)
- net A10_5V: now also U4.15 (B3), J1.19 (Pin_19), J2.21 (Pin_21); no longer U3.11 (B7)
- net A11_3V3: now also U4.4 (A2); no longer U3.8 (A6)
- net A11_5V: now also U4.16 (B2), J1.21 (Pin_21), J2.23 (Pin_23); no longer U3.12 (B6)
- net A12_3V3: now also U5.7 (A5); no longer U5.15 (B3)
- net A12_5V: now also U5.13 (B5), J2.2 (Pin_2); no longer U5.5 (A3)
- net A13_3V3: now also U5.6 (A4); no longer U3.5 (A3)
- net A13_5V: now also J3.28 (Pin_28), U5.14 (B4), J2.26 (Pin_26); no longer U3.15 (B3)
- net A14_3V3: now also U3.15 (B3); no longer U3.4 (A2)
- net A14_5V: now also U3.5 (A3), J2.27 (Pin_27); no longer U3.16 (B2)
- net A15_3V3: now also U3.14 (B4); no longer U5.16 (B2)
- net A15_5V: now also U3.6 (A4), J2.1 (Pin_1); no longer U5.4 (A2)
- net A16_3V3: now also U3.18 (B0); no longer U5.17 (B1)
- net A16_5V: now also U3.2 (A0); no longer U5.3 (A1)
- net A17_3V3: now also U3.17 (B1); no longer U3.3 (A1)
- net A17_5V: now also J3.30 (Pin_30), U3.3 (A1); no longer U3.17 (B1)
- net A18_3V3: now also U3.16 (B2); no longer U3.2 (A0)
- net A18_5V: now also U3.4 (A2); no longer U3.18 (B0)
- net A19_3V3: now also U5.8 (A6); no longer U5.18 (B0)
- net A19_5V: now also U5.12 (B6); no longer U5.2 (A0)
- net A1_3V3: now also U4.7 (A5); no longer U4.16 (B2)
- net A1_5V: now also U4.13 (B5), J1.7 (Pin_7), J2.9 (Pin_9); no longer U4.4 (A2)
- net A2_3V3: now also U5.3 (A1); no longer U4.17 (B1)
- net A2_5V: now also U5.17 (B1), J1.6 (Pin_6), J2.8 (Pin_8); no longer U4.3 (A1)
- net A3_3V3: now also U5.2 (A0); no longer U4.18 (B0)
- net A3_5V: now also U5.18 (B0), J1.5 (Pin_5), J2.7 (Pin_7); no longer U4.2 (A0)
- net A4_3V3: now also U5.5 (A3); no longer U5.11 (B7)
- net A4_5V: now also U5.15 (B3), J1.4 (Pin_4), J2.6 (Pin_6); no longer U5.9 (A7)
- net A5_3V3: now also U5.4 (A2); no longer U5.12 (B6)
- net A5_5V: now also U5.16 (B2), J1.3 (Pin_3), J2.5 (Pin_5); no longer U5.8 (A6)
- net A6_3V3: now also U4.8 (A6); no longer U5.13 (B5)
- net A6_5V: now also U4.12 (B6), J1.2 (Pin_2), J2.4 (Pin_4); no longer U5.7 (A5)
- net A7_3V3: now also U4.9 (A7); no longer U5.14 (B4)
- net A7_5V: now also U4.11 (B7), J1.1 (Pin_1), J2.3 (Pin_3); no longer U5.6 (A4)
- net A8_3V3: now also U4.3 (A1); no longer U3.6 (A4)
- net A8_5V: now also U4.17 (B1), J1.23 (Pin_23), J2.25 (Pin_25); no longer U3.14 (B4)
- net A9_3V3: now also U4.2 (A0); no longer U3.7 (A5)
- net A9_5V: now also U4.18 (B0), J1.22 (Pin_22), J2.24 (Pin_24); no longer U3.13 (B5)
- net CE_5V: now also J1.18 (Pin_18), J2.20 (Pin_20)
- net D0_3V3: now also U2.16 (B2); no longer U2.4 (A2)
- net D0_5V: now also U2.4 (A2), J1.9 (Pin_9), J2.11 (Pin_11); no longer U2.16 (B2)
- net D1_3V3: now also U2.14 (B4); no longer U2.6 (A4)
- net D1_5V: now also U2.6 (A4), J1.10 (Pin_10), J2.12 (Pin_12); no longer U2.14 (B4)
- net D2_3V3: now also U2.15 (B3); no longer U2.8 (A6)
- net D2_5V: now also U2.5 (A3), J1.11 (Pin_11), J2.13 (Pin_13); no longer U2.12 (B6)
- net D3_3V3: now also U2.13 (B5); no longer U2.9 (A7)
- net D3_5V: now also U2.7 (A5), J1.13 (Pin_13), J2.15 (Pin_15); no longer U2.11 (B7)
- net D4_3V3: now also U2.17 (B1); no longer U2.7 (A5)
- net D4_5V: now also U2.3 (A1), J1.14 (Pin_14), J2.16 (Pin_16); no longer U2.13 (B5)
- net D5_3V3: now also U2.18 (B0); no longer U2.5 (A3)
- net D5_5V: now also U2.2 (A0), J1.15 (Pin_15), J2.17 (Pin_17); no longer U2.15 (B3)
- net D6_3V3: now also U2.11 (B7); no longer U2.3 (A1)
- net D6_5V: now also U2.9 (A7), J1.16 (Pin_16), J2.18 (Pin_18); no longer U2.17 (B1)
- net D7_3V3: now also U2.12 (B6); no longer U2.2 (A0)
- net D7_5V: now also U2.8 (A6), J1.17 (Pin_17), J2.19 (Pin_19); no longer U2.18 (B0)
- net GND: now also U2.1 (A->B), U4.1 (A->B), U5.1 (A->B), J1.12 (Pin_12), J2.14 (Pin_14); no longer U3.1 (A->B)
- net OE_5V: now also J1.20 (Pin_20), J2.22 (Pin_22)
- net JP1_PWR: no longer names the net of J3.32 (Pin_32), JP1.1 (A)
- net JP1_PWR: now also J1.24 (Pin_24), J2.28 (Pin_28)
Other:
- moved on the sheet: C2, J3, JP1
